Commit message: 增加了双海康相机启动

File: src/rm_robot_description/urdf/sentry.urdf.xacro (robot description, xacro)
@@ -30,9 +30,9 @@
     <axis xyz="0 0 0" />
   </joint>
-  <link name="camera_optical_frame" />
-  <joint name="camera_optical_joint" type="fixed">
+  <link name="camera_optical_frame_first" />
+  <joint name="camera_optical_joint_first" type="fixed">
     <origin xyz="0 0 0" rpy="${-pi/2} 0 ${-pi/2}" />
     <parent link="camera_link" />
-    <child link="camera_optical_frame" />
+    <child link="camera_optical_frame_first" />
   </joint>
 </robot>
